File: converter/conv.sch (KiCad schematic (older format))
At the start: 10 parts

Commit message: part values
Parts:
- R? (x2): value 100k -> 82k
- R? (x2): value 22k -> 27k
- R? (x2): value 4k7 -> 3k3
Changed lines of the file:
@@
 LIBS:contrib
 LIBS:valves
+LIBS:conv-cache
 EELAYER 25 0
 EELAYER END
@@
 P 5000 3200
 F 0 "R?" V 4900 3150 50  0000 L CNN
-F 1 "100k" V 5100 3100 50  0000 L CNN
+F 1 "82k" V 5100 3100 50  0000 L CNN
 F 2 "" H 5000 3200 50  0000 C CNN
 F 3 "" H 5000 3200 50  0000 C CNN
@@
 P 5500 3400
 F 0 "R?" H 5600 3350 50  0000 L CNN
-F 1 "22k" H 5600 3450 50  0000 L CNN
+F 1 "27k" H 5600 3450 50  0000 L CNN
 F 2 "" H 5500 3400 50  0000 C CNN
 F 3 "" H 5500 3400 50  0000 C CNN
@@
 P 5000 4800
 F 0 "R?" V 4900 4750 50  0000 L CNN
-F 1 "100k" V 5100 4700 50  0000 L CNN
+F 1 "82k" V 5100 4700 50  0000 L CNN
 F 2 "" H 5000 4800 50  0000 C CNN
 F 3 "" H 5000 4800 50  0000 C CNN
@@
 P 5500 5000
 F 0 "R?" H 5600 4950 50  0000 L CNN
-F 1 "22k" H 5600 5050 50  0000 L CNN
+F 1 "27k" H 5600 5050 50  0000 L CNN
 F 2 "" H 5500 5000 50  0000 C CNN
 F 3 "" H 5500 5000 50  0000 C CNN
@@
 P 6900 2700
 F 0 "R?" H 7000 2650 50  0000 L CNN
-F 1 "4k7" H 7000 2750 50  0000 L CNN
+F 1 "3k3" H 7000 2750 50  0000 L CNN
 F 2 "" H 6900 2700 50  0000 C CNN
 F 3 "" H 6900 2700 50  0000 C CNN
@@
 P 6900 4300
 F 0 "R?" H 7000 4250 50  0000 L CNN
-F 1 "4k7" H 7000 4350 50  0000 L CNN
+F 1 "3k3" H 7000 4350 50  0000 L CNN
 F 2 "" H 6900 4300 50  0000 C CNN
 F 3 "" H 6900 4300 50  0000 C CNN
